File: hardware/cryosentinel.kicad_sch (KiCad schematic)
At the start: 42 parts, among them J1 USB-C-16P, J2 JST-PH-2, J3 U.FL LoRa Antenna, J4 U.FL GPS Antenna, Q1 MMBT2222, U1 ESP32-C3-MINI-1, U10 1.54in e-ink FPC-8, U11 AT25DF321, U2 SHT40, U3 ATECC608A, U4 ST25DV04K, U5 ADXL345, U6 SX1262, U7 MAX-M10S, U8 MAX17048, U9 TP4056

Commit message: fix: Correct Mermaid diagrams, restore dashboard demo image, and convert schematic to compact playlist view
Connections:
- net +3V3: no longer U1.1 (3V3), U1.2 (EN), U10.7 (Pin_7), U11.A1 (VCC), U11.B1 (~{HOLD}/IO3), U11.C2 (~{WP}/IO2), U2.5 (VDD), U2.8 (VSS), U2.9 (VSS), U8.5 (SDA)
- net +5V: no longer U9.4 (VCC), U9.8 (CE)
- net GND: no longer J1.A1 (GND), J1.A12 (GND), J1.B1 (GND), J1.B12 (GND), J2.2 (Pin_2), U1.14 (GND), U10.8 (Pin_8), U11.D2 (GND), U2.2 (ADDR), U8.2 (GND), U9.1 (TEMP), U9.3 (GND)
- net VBAT: no longer J2.1 (Pin_1), U8.1 (CELL), U9.5 (BAT)
- net BUZZER: no longer names the net of U1.11 (IO8)
- removed net CLK: U1.24 (IO20), U10.5 (Pin_5), U11.C1 (SCK)
- net CS_ADXL: no longer names the net of U1.6 (IO3)
- net CS_EINK: no longer names the net of U1.19 (IO15)
- net CS_EINK: no longer U10.4 (Pin_4)
- net CS_FLASH: no longer names the net of U1.25 (IO21)
- net CS_FLASH: no longer U11.A2 (~{CS})
- net CS_LORA: no longer names the net of U1.7 (IO4)
- net EINK_BUSY: no longer names the net of U1.16 (IO12)
- net EINK_BUSY: no longer U10.1 (Pin_1)
- net EINK_DC: no longer names the net of U1.18 (IO14)
- net EINK_DC: no longer U10.3 (Pin_3)
- net EINK_RST: no longer names the net of U1.17 (IO13)
- net EINK_RST: no longer U10.2 (Pin_2)
- net GPS_RX: no longer names the net of U1.20 (IO16)
- net GPS_TX: no longer names the net of U1.21 (IO17)
- net LED_B: no longer names the net of U1.15 (IO11)
- net LED_G: no longer names the net of U1.13 (IO10)
- net LED_R: no longer names the net of U1.12 (IO9)
- net LORA_BUSY: no longer names the net of U1.5 (IO2)
- net LORA_DIO1: no longer names the net of U1.10 (IO7)
- net LORA_RST: no longer names the net of U1.4 (IO1)
- net MISO: no longer names the net of U1.22 (IO18)
- net MISO: no longer U11.B2 (SO/IO1)
- removed net MOSI: U1.23 (IO19), U10.6 (Pin_6), U11.D1 (SI/IO0)
- removed net SCL: U1.9 (IO6), U2.4 (SCL), U8.3 (SCL)
- removed net SDA: U1.8 (IO5), U2.1 (SDA), U8.6 (~{ALRT})
- net TAMPER: no longer names the net of U1.3 (IO0)
- new net: U2.8 (VSS), U2.9 (VSS)
- new net: J1.A1 (GND), J1.A12 (GND), J1.B1 (GND), J1.B12 (GND)
- no-connect marks 125 -> 0
Other:
- note removed: "3-AXIS ACCELEROMETER"
- note removed: "BATTERY MANAGEMENT"
- note removed: "E-INK DISPLAY"
- note removed: "ESP32-C3 MCU"
- note removed: "GPS MODULE"
- note removed: "HARDWARE CRYPTO"
- note removed: "LORA MODULE"
- note removed: "NFC"
- note removed: "NOR FLASH"
- note removed: "POWER"
- note removed: "STATUS INDICATORS"
- note removed: "TEMPERATURE & HUMIDITY"
